Commit message: fix: relative paths and instructions

File: lerobot/lerobot-python/calibration/so101.urdf (robot description, URDF)
Before this commit: robot so101_new_calib, 8 links, 7 joints
Links:
- link base_link: geometry collision mesh filename=../../meshes/base_motor_holder_so101_v1.stl; collision mesh filename=../../meshes/base_so101_v2.stl
- link gripper_link: geometry collision mesh filename=../../meshes/sts3215_03a_v1.stl; collision mesh filename=../../meshes/wrist_roll_follower_so101_v1.stl
- link lower_arm_link: geometry collision mesh filename=../../meshes/motor_holder_so101_wrist_v1.stl; collision mesh filename=../../meshes/sts3215_03a_v1.stl
- link moving_jaw_so101_v1_link: geometry collision mesh filename=../../meshes/moving_jaw_so101_v1.stl; visual mesh filename=../../meshes/moving_jaw_so101_v1.stl
- link shoulder_link: geometry collision mesh filename=../../meshes/motor_holder_so101_base_v1.stl; collision mesh filename=../../meshes/rotation_pitch_so101_v1.stl
- link upper_arm_link: geometry collision mesh filename=../../meshes/sts3215_03a_v1.stl; collision mesh filename=../../meshes/upper_arm_so101_v1.stl
- link wrist_link: geometry collision mesh filename=../../meshes/sts3215_03a_no_horn_v1.stl; collision mesh filename=../../meshes/wrist_roll_pitch_so101_v2.stl
